Commit message: no more flying trees

File: server/simulation/urdf/tree.urdf (robot description, URDF)
Before this commit: robot tree, 2 links, 1 joints
Links:
- added link world
Joints:
- added joint fixed_to_ground: type fixed, parent world, child trunk

Commit message: fixing motion

File: server/simulation/urdf/tree.urdf (robot description, URDF)
Before this commit: robot tree, 2 links, 1 joints
Links:
- link trunk: geometry collision cylinder length=2.0 radius=0.1; visual cylinder length=1.0 radius=0.1
Joints:
- joint trunk_to_canopy: origin xyz=0 0 0.5 -> xyz=0 0 1.0

Commit message: Added mapping flooded areas and plotting

File: server/simulation/urdf/tree.urdf (robot description, URDF)
Before this commit: robot tree, 2 links, 1 joints
Links:
- link canopy: mass None -> 2.0
- link trunk: mass None -> 5.0; geometry collision cylinder length=1.0 radius=0.1; visual cylinder length=1.0 radius=0.1
